File: eagle/assets/layer3/Layer 3.brd (EAGLE design)
At the start: 90 x 90 mm, 82 parts, among them Q2 AO3402, X1 SM06B-SRSS-TB, Y1 8MHz

Commit message: eagle
Parts:
- moved 3U11 45.3 mm to (-7.31, 55.5), turned to 97.5 degrees
- moved 3U17 45.3 mm to (-55.5, -7.31), turned to 187.5 degrees
- moved 3U23 45.3 mm to (7.31, -55.5), turned to 277.5 degrees
- moved 3U5 45.3 mm to (55.5, 7.31), turned to 7.5 degrees
- moved 3U14 45.3 mm to (-44.4, 34.1), turned to 142.5 degrees
- moved 3U2 45.3 mm to (44.4, -34.1), turned to 322.5 degrees
- moved 3U20 45.3 mm to (-34.1, -44.4), turned to 232.5 degrees
- moved 3U8 45.3 mm to (34.1, 44.4), turned to 52.5 degrees
- moved 3U1 45.3 mm to (34.1, -44.4), turned to 307.5 degrees
- moved 3U13 45.3 mm to (-34.1, 44.4), turned to 127.5 degrees
- moved 3U19 45.3 mm to (-44.4, -34.1), turned to 217.5 degrees
- moved 3U7 45.3 mm to (44.4, 34.1), turned to 37.5 degrees
- moved 3U12 45.3 mm to (-21.4, 51.7), turned to 112.5 degrees
- moved 3U18 45.3 mm to (-51.7, -21.4), turned to 202.5 degrees
- moved 3U24 45.3 mm to (21.4, -51.7), turned to 292.5 degrees
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Other:
- board size 90 x 90 mm -> 196 x 120 mm

Commit message: eagle
Parts:
- moved BLUETOOTH 66.6 mm to (-36.1, 18.0), flipped to the top
- moved R13 55.5 mm to (2.03, 21.6), flipped to the bottom
- moved R5 47.7 mm to (10.3, 0.51), flipped to the bottom, turned to 0 degrees
- moved D1 47.0 mm to (10.0, 3.56), turned to 180 degrees
- moved R8 41.6 mm to (7.87, 12.8), flipped to the bottom, turned to 0 degrees
- moved R9 41.5 mm to (5.84, 10.7), flipped to the bottom, turned to 180 degrees
- moved R3 36.6 mm to (-12.8, 10.7), flipped to the bottom, turned to 270 degrees
- moved R7 36.1 mm to (3.94, 12.8), flipped to the bottom, turned to 180 degrees
- moved C1 36.0 mm to (-9.65, 10.7), flipped to the bottom
- moved C7 31.7 mm to (-0.25, 8.13), flipped to the bottom, turned to 270 degrees
- moved R12 30.0 mm to (-20.1, 4.57), turned to 270 degrees
- moved Y1 29.7 mm to (-0.51, 11.6), turned to 180 degrees
- moved C2 29.7 mm to (-9.65, 6.86), flipped to the bottom
- moved R6 29.6 mm to (2.92, 8.13), flipped to the bottom, turned to 270 degrees
- moved C5 29.0 mm to (-6.48, 10.7), flipped to the bottom, turned to 270 degrees
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Other:
- outline, holes or cut-outs redrawn

Commit message: cancer pain in the ass
Parts:
- moved BLUETOOTH 67.7 mm to (30.5, 30.1)
- moved X1 61.6 mm to (0.03, 44.1), turned to 0 degrees
- moved 4TH_LAYER 55.8 mm to (-10.9, 43.8), turned to 0 degrees
- moved 5V_PWR 44.6 mm to (-29.0, 12.3)
- moved U$14 38.3 mm to (-15.4, 13.2)
- moved C3 36.5 mm to (5.49, 40.2), turned to 0 degrees
- moved C1 35.6 mm to (13.1, 38.1), turned to 0 degrees
- moved C2 34.6 mm to (5.49, 38.0), turned to 0 degrees
- moved R5 32.2 mm to (-20.3, 10.7), flipped to the top, turned to 180 degrees
- moved D1 31.9 mm to (-20.3, 13.5)
- moved R6 27.1 mm to (6.35, 35.0), turned to 90 degrees
- moved C5 26.5 mm to (3.99, 35.0), turned to 90 degrees
- moved R9 25.6 mm to (14.0, 35.0), turned to 90 degrees
- moved Y1 24.1 mm to (0.36, -12.6), turned to 0 degrees
- moved S1 22.9 mm to (10.2, 24.2), turned to 0 degrees
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Routing:
- net 5V_SWITCH: track 0.00 -> 93.7 mm
- net 3V3_SWITCH: track 0.00 -> 88.5 mm, vias 0 -> 7
- net MOSI: track 0.00 -> 84.9 mm
- net RX1_ST2: track 0.00 -> 80.7 mm, vias 0 -> 1
- net MISO: track 0.00 -> 79.3 mm, vias 0 -> 2
- net SDA0_TEE: track 0.00 -> 79.3 mm
- net TX1_ST2: track 0.00 -> 78.0 mm
- net SWCLK: track 0.00 -> 75.0 mm, vias 0 -> 2
- net SCL0_TEE: track 0.00 -> 73.1 mm
- net RESET: track 0.00 -> 73.1 mm, vias 0 -> 3
- net SCK: track 0.00 -> 67.8 mm, vias 0 -> 1
- net ESC_LV: track 0.00 -> 67.4 mm, vias 0 -> 2
- net 3.3V: track 0.00 -> 54.4 mm, vias 0 -> 1
- net SWDIO: track 0.00 -> 49.2 mm, vias 0 -> 4
- net TX3_ST1: track 0.00 -> 46.2 mm
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- added copper zone on layer 1, net GND
- added copper zone on layer 16, net GND
Other:
- outline, holes or cut-outs redrawn

Commit message: shi
Parts:
- moved U$14 26.0 mm to (-19.9, 38.8)
- moved Y1 8.31 mm to (0.76, -20.9)
- moved C6 6.81 mm to (2.00, -15.6)
- moved C7 6.81 mm to (-0.44, -15.6)
- moved BOOT 1.36 mm to (-29.0, 4.61)
- moved R12 1.32 mm to (-18.9, 5.21)
- moved R4 0.41 mm to (-31.2, 1.11)
Routing:
- net 3V3_SWITCH: track 88.5 -> 689.5 mm, vias 7 -> 9
- net IR20: track 0.00 -> 99.1 mm
- net IR21: track 0.00 -> 98.1 mm, vias 0 -> 1
- net IR12: track 0.00 -> 91.0 mm, vias 0 -> 6
- net IR8: track 0.00 -> 91.0 mm, vias 0 -> 2
- net IR22: track 0.00 -> 83.1 mm, vias 0 -> 2
- net IR7: track 0.00 -> 80.1 mm, vias 0 -> 2
- net IR9: track 0.00 -> 76.9 mm, vias 0 -> 2
- net IR17: track 0.00 -> 76.2 mm, vias 0 -> 2
- net IR6: track 0.00 -> 74.6 mm, vias 0 -> 2
- net IR5: track 0.00 -> 72.2 mm, vias 0 -> 2
- net IR14: track 0.00 -> 71.4 mm, vias 0 -> 2
- net IR18: track 0.00 -> 69.5 mm
- net IR23: track 0.00 -> 68.7 mm, vias 0 -> 2
- net IR4: track 0.00 -> 68.4 mm, vias 0 -> 2
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
Commit message: edit
Routing:
- net BOOT0: track 23.2 -> 42.7 mm, vias 5 -> 7
- net SCK: track 47.2 -> 48.7 mm
Changed lines of the file:
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@@
 </layers>
 <board>
-<fusionsync huburn="a.YnVzaW5lc3M6Z21haWwxNDMxNzc3" projecturn="a.YnVzaW5lc3M6Z21haWwxNDMxNzc3IzIwMjEwMTE1MzcxOTY3NzA2" f3durn="urn:adsk.wipprod:dm.lineage:aVCnS0wBSYmPTEc4_Ognuw" pcbguid="" lastpulledtime="2021-11-29T07:02:40Z" lastsyncedchangeguid="" latestrevisionid="36314339-9404-4f6b-9740-392bf09eeaae" lastsyncedrevisionid="6d987efc-c976-4d24-83f3-6c011a708b88" lastboardhashguid="6a7cd929-a916-b77f-e957-806ddc053c05" lastpushedtime="2021-11-26T17:01:38Z" linktopcb3d="true"/>
+<fusionsync huburn="a.YnVzaW5lc3M6Z21haWwxNDMxNzc3" projecturn="a.YnVzaW5lc3M6Z21haWwxNDMxNzc3IzIwMjEwMTE1MzcxOTY3NzA2" f3durn="urn:adsk.wipprod:dm.lineage:aVCnS0wBSYmPTEc4_Ognuw" pcbguid="" lastpulledtime="2021-11-29T07:02:40Z" lastsyncedchangeguid="" latestrevisionid="601b6d08-ecd5-4038-aac2-37d21264e25e" lastsyncedrevisionid="601b6d08-ecd5-4038-aac2-37d21264e25e" lastboardhashguid="b4fabb40-d086-cded-99aa-3d99f0dd81bb" lastpushedtime="2021-11-30T15:03:43Z" linktopcb3d="true"/>
 <plain>
 <hole x="-14.478" y="5.588" drill="3"/>
@@
 <wire x1="-31.215" y1="1.9612" x2="-29.4388" y2="1.9612" width="0.254" layer="1"/>
 <wire x1="-29.4388" y1="1.9612" x2="-29.04" y2="2.36" width="0.254" layer="1"/>
-<wire x1="4.8088" y1="-1.3262" x2="-13.4" y2="-4.5" width="0" layer="19" extent="1-16"/>
 <wire x1="-29.04" y1="2.36" x2="-28.208" y2="2.36" width="0.254" layer="1"/>
 <wire x1="-28.208" y1="2.36" x2="-27.648" y2="1.8" width="0.254" layer="1"/>
@@
 <via x="-20.8" y="-3.28" extent="1-16" drill="0.508"/>
 <wire x1="-20.8" y1="-3.28" x2="-19.68" y2="-4.4" width="0.254" layer="1"/>
-<wire x1="-19.68" y1="-4.4" x2="-14.3" y2="-4.4" width="0.254" layer="1"/>
-<wire x1="-14.3" y1="-4.4" x2="-13.5" y2="-4.4" width="0.254" layer="1"/>
+<wire x1="-19.68" y1="-4.4" x2="-13.5" y2="-4.4" width="0.254" layer="1"/>
 <wire x1="-13.5" y1="-4.4" x2="-13.4" y2="-4.5" width="0.254" layer="1"/>
 <via x="-13.4" y="-4.5" extent="1-16" drill="0.508"/>
+<wire x1="4.8088" y1="-1.3262" x2="-0.08" y2="-1.3262" width="0.2032" layer="16"/>
+<wire x1="-0.08" y1="-1.3262" x2="-0.1" y2="-1.3462" width="0.2032" layer="16"/>
+<via x="-0.1" y="-1.3462" extent="1-16" drill="0.508"/>
+<via x="-7.66" y="-4.49" extent="1-16" drill="0.508"/>
+<wire x1="-0.1" y1="-1.3462" x2="-1.8102" y2="-3.0564" width="0.2032" layer="1"/>
+<wire x1="-1.8102" y1="-3.0564" x2="-3.22960625" y2="-3.0564" width="0.2032" layer="1"/>
+<wire x1="-4.66320625" y1="-4.49" x2="-7.66" y2="-4.49" width="0.2032" layer="1"/>
+<wire x1="-3.22960625" y1="-3.0564" x2="-4.66320625" y2="-4.49" width="0.2032" layer="1"/>
+<wire x1="-7.66" y1="-4.49" x2="-7.67" y2="-4.5" width="0.2032" layer="16"/>
+<wire x1="-7.67" y1="-4.5" x2="-13.4" y2="-4.5" width="0.2032" layer="16"/>
 </signal>
 <signal name="N$72">
@@
 <wire x1="-45.45163125" y1="-31.6" x2="-45.772528125" y2="-31.920896875" width="0.254" layer="16"/>
 <wire x1="-40.6" y1="-31.6" x2="-45.45163125" y2="-31.6" width="0.254" layer="16"/>
-<wire x1="-14.908" y1="-15.348" x2="-2.46" y2="-2.9" width="0.254" layer="1"/>
-<wire x1="-2.46" y1="-2.9" x2="0.4" y2="-2.9" width="0.254" layer="1"/>
-<wire x1="0.4" y1="-2.9" x2="1" y2="-2.3" width="0.254" layer="1"/>
+<wire x1="-14.908" y1="-15.348" x2="-3.05" y2="-3.49" width="0.254" layer="1"/>
+<wire x1="-3.05" y1="-3.49" x2="-0.19" y2="-3.49" width="0.254" layer="1"/>
+<wire x1="-0.19" y1="-3.49" x2="1" y2="-2.3" width="0.254" layer="1"/>
 <wire x1="1" y1="-2.3" x2="1" y2="0.56" width="0.254" layer="1"/>
 </signal>
@@
 <wire x1="-1.27" y1="16.51" x2="-1.27" y2="8.31794375" width="0.254" layer="1"/>
 <wire x1="-1.27" y1="8.31794375" x2="-4.44" y2="5.14794375" width="0.254" layer="1"/>
-<wire x1="-4.44" y1="-3.69205625" x2="-9.423971875" y2="-8.676028125" width="0.254" layer="1"/>
-<wire x1="-4.44" y1="5.14794375" x2="-4.44" y2="-3.69205625" width="0.254" layer="1"/>
+<wire x1="-4.44" y1="-1" x2="-4.44" y2="5.14794375" width="0.254" layer="1"/>
 <wire x1="-9.423971875" y1="-8.676028125" x2="-9.423971875" y2="-20.084971875" width="0.254" layer="16"/>
 <wire x1="-9.423971875" y1="-20.084971875" x2="-10.439" y2="-21.1" width="0.254" layer="16"/>
@@
 <wire x1="-10.439" y1="-21.1" x2="-10.675" y2="-21.336" width="0.254" layer="1"/>
 <wire x1="-10.675" y1="-21.336" x2="-16.129" y2="-21.336" width="0.254" layer="1"/>
+<wire x1="-9.423971875" y1="-8.676028125" x2="-9.423971875" y2="-5.023971875" width="0.2032" layer="1"/>
+<wire x1="-7.5" y1="-3.1" x2="-5" y2="-3.1" width="0.2032" layer="1"/>
+<wire x1="-5" y1="-3.1" x2="-4.44" y2="-2.54" width="0.2032" layer="1"/>
+<wire x1="-4.44" y1="-2.54" x2="-4.44" y2="-1" width="0.2032" layer="1"/>
+<wire x1="-9.423971875" y1="-5.023971875" x2="-7.5" y2="-3.1" width="0.2032" layer="1"/>
 </signal>
 <signal name="SS">

Commit message: done with layer 4
Routing:
- net 5V_SWITCH: track 119.1 -> 113.4 mm, vias 4 -> 3
- net 5V: track 26.3 -> 23.4 mm

Commit message: changes to layout in layer 3
Parts:
- moved U$8 80.7 mm to (17.8, 36.8), turned to 180 degrees
- moved BLUETOOTH 71.0 mm to (-14.0, -25.2), turned to 90 degrees
- moved R8 55.0 mm to (-25.4, -5.84), flipped to the top
- moved R6 55.0 mm to (-30.5, -5.82), flipped to the top
- moved R9 55.0 mm to (-22.9, -5.85), flipped to the top
- moved R7 55.0 mm to (-28.0, -5.82), flipped to the top
- moved S1 53.0 mm to (-26.7, -14.0)
- moved R5 51.0 mm to (19.1, 43.2)
- moved Y1 50.1 mm to (0.00, 29.2), turned to 180 degrees
- moved 5V_PWR 49.4 mm to (20.1, 7.85), turned to 0 degrees
- moved C6 48.8 mm to (-2.54, 33.0), turned to 0 degrees
- moved C7 48.6 mm to (1.27, 33.0), turned to 0 degrees
- moved D1 48.5 mm to (19.0, 41.9)
- moved 3V3_PWR 47.4 mm to (-38.6, 1.89), turned to 180 degrees
- moved R4 45.4 mm to (11.9, -13.1), turned to 270 degrees
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Routing:
- net 3V3_SWITCH: track 689.5 -> 0.00 mm, vias 9 -> 0
- net 3.3V: track 118.9 -> 0.00 mm, vias 8 -> 0
- net ESC_LV: track 118.8 -> 0.00 mm, vias 9 -> 0
- net 5V_SWITCH: track 113.4 -> 0.00 mm, vias 3 -> 0
- net IR20: track 99.1 -> 0.00 mm
- net MISO: track 98.4 -> 0.00 mm, vias 12 -> 0
- net IR21: track 98.1 -> 0.00 mm, vias 1 -> 0
- net MOSI: track 92.9 -> 0.00 mm, vias 3 -> 0
- net TX1_ST2: track 91.9 -> 0.00 mm, vias 3 -> 0
- net IR12: track 91.0 -> 0.00 mm, vias 6 -> 0
- net IR8: track 91.0 -> 0.00 mm, vias 2 -> 0
- net RX1_ST2: track 89.4 -> 0.00 mm, vias 2 -> 0
- net IR22: track 83.1 -> 0.00 mm, vias 2 -> 0
- net IR7: track 80.1 -> 0.00 mm, vias 2 -> 0
- net IR9: track 76.9 -> 0.00 mm, vias 2 -> 0
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Other:
- outline, holes or cut-outs redrawn

Commit message: eagle
Parts:
- moved U$14 15.3 mm to (-37.7, 9.36), turned to 90 degrees
- moved 3C20 13.6 mm to (6.38, -50.6), flipped to the bottom, turned to 7 degrees
- moved 3C15 13.5 mm to (-47.3, -19.1), flipped to the bottom, turned to 0 degrees
- moved 3C21 13.5 mm to (19.1, -47.3), flipped to the bottom, turned to 0 degrees
- moved 3C3 13.5 mm to (47.3, 19.1), flipped to the bottom, turned to 0 degrees
- moved 3C9 13.5 mm to (-19.1, 47.3), flipped to the bottom, turned to 0 degrees
- moved 3C1 13.5 mm to (50.5, -7.10), flipped to the bottom, turned to 0 degrees
- moved 3C13 13.5 mm to (-50.5, 7.10), flipped to the bottom, turned to 0 degrees
- moved 3C19 13.5 mm to (-7.10, -50.5), flipped to the bottom, turned to 0 degrees
- moved 3C7 13.5 mm to (7.10, 50.5), flipped to the bottom, turned to 0 degrees
- moved 3C11 13.5 mm to (-40.2, 31.4), flipped to the bottom, turned to 0 degrees
- moved 3C17 13.5 mm to (-31.4, -40.2), flipped to the bottom, turned to 0 degrees
- moved 3C23 13.5 mm to (40.2, -31.4), flipped to the bottom, turned to 0 degrees
- moved 3C5 13.5 mm to (31.4, 40.2), flipped to the bottom, turned to 0 degrees
- moved 3C14 13.5 mm to (-50.6, -6.22), flipped to the bottom, turned to 0 degrees
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