File: eagle/assets/layer3/Layer 3.sch (EAGLE design)
At the start: 84 parts, among them Q2 AO3402, X1 SM06B-SRSS-TB, Y1 8MHz

Commit message: Edited cura
Parts:
- removed COMPASS: BNO055, JH:BNO055
- added BNO055: (no value), SparkFun-Connectors:CONN_08LOCK
Connections:
- net 3V3_SWITCH: now also BNO055.8; no longer COMPASS.VCC
- net GND: now also BNO055.7; no longer COMPASS.GND
- net SCL1: now also BNO055.5; no longer COMPASS.SCL
- net SDA1: now also BNO055.6; no longer COMPASS.SDA
Changed lines of the file:
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@@
 <layer number="56" name="wert" color="7" fill="1" visible="no" active="no"/>
 <layer number="57" name="tCAD" color="7" fill="1" visible="no" active="no"/>
+<layer number="58" name="bCAD" color="7" fill="1" visible="no" active="no"/>
 <layer number="59" name="tCarbon" color="7" fill="1" visible="no" active="no"/>
 <layer number="60" name="bCarbon" color="7" fill="1" visible="no" active="no"/>
@@
 <layer number="250" name="Descript" color="3" fill="1" visible="no" active="no"/>
 <layer number="251" name="SMDround" color="12" fill="11" visible="no" active="no"/>
+<layer number="253" name="Extra" color="7" fill="1" visible="no" active="no"/>
 <layer number="254" name="cooling" color="7" fill="1" visible="no" active="no"/>
 <layer number="255" name="routoute" color="7" fill="1" visible="no" active="no"/>
@@
 <part name="J1" library="Connectors" library_urn="urn:adsk.eagle:library:19813715" deviceset="CONN_02" device="LOCK" package3d_urn="urn:adsk.eagle:package:19813850/2"/>
 <part name="FRAME7" library="SparkFun-Aesthetics" library_urn="urn:adsk.eagle:library:507" deviceset="FRAME-A4L" device=""/>
-<part name="COMPASS" library="JH" library_urn="urn:adsk.eagle:library:6027132" deviceset="BNO055" device="" package3d_urn="urn:adsk.eagle:package:16833735/3"/>
 <part name="SUPPLY4" library="SparkFun-PowerSymbols" deviceset="3.3V" device=""/>
 <part name="SUPPLY5" library="SparkFun-PowerSymbols" deviceset="3.3V" device=""/>
@@
 <part name="TEENSY4" library="Teensy-4.0" deviceset="TEENSY-4.0-FULL-BREAKOUT-PINS" device=""/>
 <part name="GND35" library="SparkFun-PowerSymbols" library_urn="urn:adsk.eagle:library:530" deviceset="GND" device=""/>
+<part name="BNO055" library="SparkFun-Connectors" deviceset="CONN_08" device="LOCK"/>
 </parts>
 <sheets>
@@
 <attribute name="SHEET" x="200.66" y="6.35" size="2.54" layer="94" font="vector"/>
 </instance>
-<instance part="COMPASS" gate="G$1" x="106.68" y="106.68" smashed="yes">
-<attribute name="NAME" x="101.6" y="117.348" size="1.27" layer="95"/>
-</instance>
 <instance part="SUPPLY4" gate="G$1" x="175.26" y="109.22" smashed="yes" rot="R270">
 <attribute name="VALUE" x="178.054" y="109.22" size="1.778" layer="96" rot="R270" align="bottom-center"/>
@@
 <instance part="GND34" gate="1" x="138.938" y="111.76" smashed="yes" rot="R90">
 <attribute name="VALUE" x="141.732" y="111.76" size="1.778" layer="96" rot="R270" align="top-center"/>
+</instance>
+<instance part="BNO055" gate="G$1" x="114.3" y="104.14" smashed="yes">
+<attribute name="VALUE" x="109.22" y="91.694" size="1.778" layer="96" font="vector"/>
+<attribute name="NAME" x="109.22" y="117.348" size="1.778" layer="95" font="vector"/>
 </instance>
 </instances>
@@
 <net name="3V3_SWITCH" class="0">
 <segment>
-<pinref part="COMPASS" gate="G$1" pin="VCC"/>
 <wire x1="119.38" y1="114.3" x2="121.92" y2="114.3" width="0.1524" layer="91"/>
 <wire x1="121.92" y1="114.3" x2="121.92" y2="119.38" width="0.1524" layer="91"/>
 <label x="116.84" y="119.38" size="1.778" layer="95"/>
+<pinref part="BNO055" gate="G$1" pin="8"/>
 </segment>
 </net>
@@
 <net name="GND" class="0">
 <segment>
-<pinref part="COMPASS" gate="G$1" pin="GND"/>
 <wire x1="119.38" y1="111.76" x2="136.398" y2="111.76" width="0.1524" layer="91"/>
 <pinref part="GND34" gate="1" pin="GND"/>
+<pinref part="BNO055" gate="G$1" pin="7"/>
 </segment>
 </net>
 <net name="SDA1" class="0">
 <segment>
-<pinref part="COMPASS" gate="G$1" pin="SDA"/>
 <wire x1="119.38" y1="109.22" x2="132.08" y2="109.22" width="0.1524" layer="91"/>
 <label x="119.38" y="109.22" size="1.778" layer="95"/>
+<pinref part="BNO055" gate="G$1" pin="6"/>
 </segment>
 <segment>
@@
 <net name="SCL1" class="0">
 <segment>
-<pinref part="COMPASS" gate="G$1" pin="SCL"/>
 <wire x1="119.38" y1="106.68" x2="132.08" y2="106.68" width="0.1524" layer="91"/>
 <label x="119.38" y="106.68" size="1.778" layer="95"/>
-</segment>
-<segment>
+<pinref part="BNO055" gate="G$1" pin="5"/>
+</segment>
+<segment>
