File: eagle/assets/layer4/layer4.brd (EAGLE design)
At the start: 102.9 x 102.9 mm, 45 parts, among them Y1 8MHz

Commit message: more shit need to do
Parts:
- moved R2 29.7 mm to (-30.6, 3.39), turned to 270 degrees
- moved D1 16.8 mm to (-16.4, -22.3), turned to 270 degrees
- moved R4 12.3 mm to (-5.60, -25.6), flipped to the bottom
- moved R5 2.48 mm to (-14.3, -22.2), turned to 270 degrees
Routing:
- net N$70: track 30.7 -> 1.65 mm, vias 2 -> 0
- net N$74: track 25.7 -> 2.08 mm, vias 2 -> 0
- net 3V3_SWITCH: track 103.5 -> 110.5 mm, vias 6 -> 5
- net RESET: track 51.9 -> 45.1 mm
- net GND: track 0.00 -> 5.65 mm, vias 0 -> 1
- net SWCLK: track 27.9 -> 32.5 mm
- net L3R: track 14.4 -> 10.2 mm
- net SWDIO: track 26.1 -> 27.8 mm
- net N$73: track 26.4 -> 27.4 mm
- net BOOT0: track 53.8 -> 54.6 mm
- net OSC_OUT: track 26.7 -> 27.4 mm
- net N$24: track 186.9 -> 187.5 mm
- net L2R: track 13.2 -> 13.7 mm
- net L2C: track 9.15 -> 9.39 mm, vias 2 -> 0

Commit message: about done
Parts:
- moved 1R5 10.9 mm to (28.7, -22.9), flipped to the bottom, turned to 180 degrees
- moved C1 8.09 mm to (8.57, -24.0)
- moved C3 8.09 mm to (4.13, -24.0)
- moved C2 8.09 mm to (6.38, -24.0)
- moved 3RD_LAYER 5.87 mm to (26.3, -7.67), turned to 270 degrees
Routing:
- net RX2: track 25.9 -> 8.56 mm, vias 2 -> 1
- net N$11: track 202.2 -> 189.0 mm, vias 7 -> 4
- net L1C: track 21.6 -> 33.4 mm, vias 2 -> 3
- net TX2: track 27.7 -> 20.8 mm
- net 3V3_SWITCH: track 110.5 -> 104.8 mm
- net 3.3V: track 69.0 -> 65.3 mm
- net N$21: track 99.6 -> 102.8 mm
- net N$23: track 185.4 -> 182.7 mm
- net N$22: track 220.7 -> 218.9 mm
- net BOOT0: track 54.6 -> 52.8 mm
- net L3C: track 16.5 -> 15.0 mm, vias 2 -> 0
- net L4C: track 24.5 -> 23.3 mm
- net RESET: track 45.1 -> 45.9 mm

Commit message: done with layer 4
Parts:
- removed BNO_RESET: MOMENTARY_SWITCH_4X3, MY-LIBRARY:MOMENTARY_SWITCH_4X3
- added COMPASS_RST: MOMENTARY_SWITCH_4X3, MY-LIBRARY:MOMENTARY_SWITCH_4X3
- moved 3V3_PWR 44.4 mm to (15.3, 2.17), turned to 90 degrees
- moved 3RD_LAYER 11.5 mm to (15.2, -4.62)
- moved 1R4 6.06 mm to (-3.49, -10.4)
- moved 1R6 4.33 mm to (17.2, -19.6), turned to 270 degrees
- moved BOOT 4.07 mm to (-26.7, -6.61)
- moved C2 1.84 mm to (8.22, -24.1)
- moved C3 1.84 mm to (5.97, -24.0)
- moved C1 1.84 mm to (10.4, -24.0)
- moved R3 1.77 mm to (-14.7, -16.6)
- moved R1 0.80 mm to (-11.9, -16.6)
- moved 1R2 0.59 mm to (-9.93, -28.6)
- moved C5 0.10 mm to (-8.87, -16.6)
Connections:
- net BNO_RST: now also COMPASS_RST.P$2; no longer BNO_RESET.P$2
- net GND: now also COMPASS_RST.P$1; no longer BNO_RESET.P$1
Routing:
- net 3.3V: track 65.3 -> 5.43 mm
- net 3V3_SWITCH: track 104.8 -> 114.4 mm
- net N$21: track 102.8 -> 96.5 mm
- net N$22: track 218.9 -> 213.8 mm
- net TX2: track 20.8 -> 15.8 mm, vias 2 -> 0
- net RX2: track 8.56 -> 13.5 mm, vias 1 -> 0
- net L4R: track 6.84 -> 2.50 mm
- net BOOT0: track 52.8 -> 48.8 mm
- net N$72: track 27.5 -> 25.5 mm
- net L2C: track 9.39 -> 11.2 mm, vias 0 -> 2
- net SWCLK: track 32.5 -> 33.4 mm
- net SWDIO: track 27.9 -> 27.1 mm

Commit message: ??
Other:
- board size 102.9 x 102.9 mm -> 197 x 149.4 mm
Changed lines of the file:
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@@
 <board>
 <plain>
-<circle x="0" y="0" radius="51.441709375" width="0.001" layer="20"/>
 <circle x="0" y="0" radius="1.6" width="0.001" layer="20"/>
 <circle x="0" y="-45" radius="1.6" width="0.001" layer="20"/>
@@
 <circle x="0" y="-45" radius="3.54114375" width="0.1524" layer="39"/>
 <circle x="-45" y="0" radius="3.54114375" width="0.1524" layer="39"/>
+<circle x="93.998990625" y="-0.435540625" radius="1.6" width="0.001" layer="20"/>
+<circle x="0" y="0" radius="1.6" width="0.001" layer="20"/>
+<circle x="-0.43323125" y="-93.499" radius="1.6" width="0.001" layer="20"/>
+<circle x="-93.998990625" y="0.435540625" radius="1.6" width="0.001" layer="20"/>
+<wire x1="-95.326390625" y1="-3.66913125" x2="-96.427240625" y2="-3.35308125" width="0.001" layer="20" curve="-33.28"/>
+<wire x1="-96.427240625" y1="-3.35308125" x2="-93.978140625" y2="4.935490625" width="0.001" layer="20" curve="-147.61"/>
+<wire x1="-93.978140625" y1="4.935490625" x2="-40.97853125" y2="31.09678125" width="0.001" layer="20" curve="53.07"/>
+<wire x1="-40.97853125" y1="31.09678125" x2="41.264940625" y2="30.715709375" width="0.001" layer="20" curve="-106.14"/>
+<wire x1="41.264940625" y1="30.715709375" x2="94.019840625" y2="4.064409375" width="0.001" layer="20" curve="53.07"/>
+<wire x1="94.019840625" y1="4.064409375" x2="96.39201875" y2="-4.2465" width="0.001" layer="20" curve="-147.61"/>
+<wire x1="96.39201875" y1="-4.2465" x2="95.2883" y2="-4.552340625" width="0.001" layer="20" curve="-33.28"/>
+<wire x1="95.2883" y1="-4.552340625" x2="4.06651875" y2="-93.54716875" width="0.001" layer="20" curve="90.88"/>
+<wire x1="4.06651875" y1="-93.54716875" x2="-4.93321875" y2="-93.50546875" width="0.001" layer="20" curve="-179.3"/>
+<wire x1="-4.93321875" y1="-93.50546875" x2="-95.326390625" y2="-3.66913125" width="0.001" layer="20" curve="90.88"/>
+<circle x="93.974" y="-0.35" radius="3.54114375" width="0.1524" layer="39"/>
+<circle x="-94.026" y="0.45" radius="3.54114375" width="0.1524" layer="39"/>
 </plain>
 <attributes>
