File: eagle/assets/layer4/layer4.brd (EAGLE design)
At the start: 197 x 149.4 mm, 45 parts, among them Y1 8MHz

Commit message: Fixed more stuff
Routing:
- net RX2: track 45.3 -> 46.8 mm
- net N$23: track 182.7 -> 183.9 mm
- net N$24: track 187.5 -> 186.5 mm
- net N$20: track 72.1 -> 71.4 mm
- net N$19: track 108.0 -> 108.5 mm
- net GND: vias 1 -> 3

Commit message: Fixed more stuff
Routing:
- net N$73: track 31.5 -> 30.6 mm
Changed lines of the file:
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@@
 </layers>
 <board>
-<fusionsync huburn="a.YnVzaW5lc3M6Z21haWwxNDMxNzc3" projecturn="a.YnVzaW5lc3M6Z21haWwxNDMxNzc3IzIwMjIwMTE1NDg1NTYyMzgx" f3durn="urn:adsk.wipprod:dm.lineage:GR2y0BrRQ0CTRm3otW2Crg" pcbguid="" lastpulledtime="" lastsyncedchangeguid="" latestrevisionid="3192f427-fcfb-4659-9816-bf69bf25f697" lastsyncedrevisionid="3192f427-fcfb-4659-9816-bf69bf25f697" lastboardhashguid="d540677b-a4e6-8d71-c3d2-ac2cbcd7b6df" lastpushedtime="2022-02-21T14:17:24Z" linktopcb3d="true"/>
+<fusionsync huburn="a.YnVzaW5lc3M6Z21haWwxNDMxNzc3" projecturn="a.YnVzaW5lc3M6Z21haWwxNDMxNzc3IzIwMjIwMTE1NDg1NTYyMzgx" f3durn="urn:adsk.wipprod:dm.lineage:GR2y0BrRQ0CTRm3otW2Crg" pcbguid="" lastpulledtime="" lastsyncedchangeguid="" latestrevisionid="8fda0457-b0fc-4104-8fa0-cd10d9f43d4e" lastsyncedrevisionid="8fda0457-b0fc-4104-8fa0-cd10d9f43d4e" lastboardhashguid="5e6a0963-015a-74ec-4e78-739dcc087a8e" lastpushedtime="2022-02-21T14:24:05Z" linktopcb3d="true"/>
 <plain>
 <circle x="-7.874" y="-6.35" radius="3.54114375" width="0.1524" layer="39"/>
@@
 <contactref element="1R3" pad="2"/>
 <contactref element="STM32" pad="26"/>
-<wire x1="-12.832" y1="-12.599" x2="-11.601" y2="-12.599" width="0.254" layer="1"/>
-<wire x1="-11.601" y1="-12.599" x2="-11.4" y2="-12.8" width="0.254" layer="1"/>
-<via x="-11.4" y="-12.8" extent="1-16" drill="0.508"/>
-<wire x1="-11.4" y1="-12.8" x2="-10.317" y2="-13.883" width="0.254" layer="16"/>
-<wire x1="-10.317" y1="-13.883" x2="-5.41101875" y2="-13.883" width="0.254" layer="16"/>
+<wire x1="-12.832" y1="-12.599" x2="-10.332" y2="-12.599" width="0.254" layer="1"/>
+<wire x1="-10.332" y1="-12.599" x2="-10.309" y2="-12.622" width="0.254" layer="1"/>
+<via x="-10.309" y="-12.622" extent="1-16" drill="0.508"/>
+<wire x1="-10.309" y1="-12.622" x2="-9.048" y2="-13.883" width="0.254" layer="16"/>
+<wire x1="-9.048" y1="-13.883" x2="-5.41101875" y2="-13.883" width="0.254" layer="16"/>
 <wire x1="-5.41101875" y1="-13.883" x2="-5.2332" y2="-13.70518125" width="0.254" layer="16"/>
 <via x="-5.2332" y="-13.70518125" extent="1-16" drill="0.508"/>
@@
 <wire x1="1.0152" y1="-8.987225" x2="0.091975" y2="-8.064" width="0.254" layer="1"/>
 <wire x1="-3.243" y1="-8.064" x2="0.091975" y2="-8.064" width="0.254" layer="1"/>
-<wire x1="-12.4618" y1="-22.4678" x2="-12.4618" y2="-10.8618" width="0.254" layer="16"/>
+<wire x1="-12.4618" y1="-22.4678" x2="-11.9458" y2="-21.9518" width="0.254" layer="16"/>
+<wire x1="-11.9458" y1="-11.8958" x2="-11.9458" y2="-21.9518" width="0.254" layer="16"/>
 <wire x1="-14.31" y1="-23.091" x2="-13.085" y2="-23.091" width="0.254" layer="1"/>
 <wire x1="-13.085" y1="-23.091" x2="-12.4618" y2="-22.4678" width="0.254" layer="1"/>
 <via x="-12.4618" y="-22.4678" extent="1-16" drill="0.508"/>
-<wire x1="-12.4618" y1="-10.8618" x2="-11.7" y2="-10.1" width="0.254" layer="16"/>
+<wire x1="-11.9458" y1="-11.8958" x2="-10.15" y2="-10.1" width="0.254" layer="16"/>
 <wire x1="-3.887" y1="-8.064" x2="-3.243" y2="-8.064" width="0.254" layer="16"/>
 <wire x1="-3.887" y1="-8.064" x2="-5.923" y2="-10.1" width="0.254" layer="16"/>
 <via x="-3.243" y="-8.064" extent="1-16" drill="0.508"/>
-<wire x1="-11.7" y1="-10.1" x2="-5.923" y2="-10.1" width="0.254" layer="16"/>
+<wire x1="-10.15" y1="-10.1" x2="-5.923" y2="-10.1" width="0.254" layer="16"/>
 </signal>
 <signal name="N$74">
@@
 <wire x1="-23.285" y1="2.545" x2="-21.958" y2="1.218" width="0.254" layer="1"/>
 <via x="-21.958" y="1.218" extent="1-16" drill="0.508"/>
-<wire x1="-21.958" y1="1.218" x2="-13.3" y2="-7.44" width="0.254" layer="16"/>
-<wire x1="-13.3" y1="-7.44" x2="-13.3" y2="-16.892" width="0.254" layer="16"/>
-<via x="-13.3" y="-16.892" extent="1-16" drill="0.508"/>
-<wire x1="-13.3" y1="-16.892" x2="-11.922" y2="-16.892" width="0.254" layer="1"/>
-<wire x1="-11.922" y1="-16.892" x2="-11.92" y2="-16.89" width="0.254" layer="1"/>
+<wire x1="-21.958" y1="1.218" x2="-13.422" y2="-7.318" width="0.254" layer="16"/>
+<wire x1="-13.422" y1="-7.318" x2="-13.422" y2="-17.103" width="0.254" layer="16"/>
+<via x="-13.422" y="-17.103" extent="1-16" drill="0.508"/>
+<wire x1="-13.422" y1="-17.103" x2="-12.133" y2="-17.103" width="0.254" layer="1"/>
+<wire x1="-12.133" y1="-17.103" x2="-11.92" y2="-16.89" width="0.254" layer="1"/>
 <wire x1="-11.92" y1="-16.89" x2="-10.51" y2="-16.89" width="0.254" layer="1"/>
 <wire x1="-10.51" y1="-16.89" x2="-10.5" y2="-16.9" width="0.254" layer="1"/>

Commit message: Final Check
Parts:
- moved 1R5 26.1 mm to (4.10, -31.5)
Routing:
- net L1C: track 33.4 -> 11.4 mm, vias 3 -> 1
- net N$11: track 188.5 -> 197.2 mm
- net N$22: track 214.3 -> 212.7 mm
- net N$23: track 183.9 -> 183.2 mm

Commit message: Edited Layer 4
Parts:
- removed COMPASS_RST: MOMENTARY_SWITCH_4X3, MY-LIBRARY:MOMENTARY_SWITCH_4X3
- added R6, R7: 4.7k, SparkFun-Resistors:0603
Connections:
- removed net BNO_RST: COMPASS.2, COMPASS_RST.P$2, STM32.18
- net 3.3V: now also R6.2, R7.2
- net GND: no longer COMPASS.4, COMPASS_RST.P$1
- net SCL2: now also R7.1, STM32.21
- net SDA2: now also R6.1, STM32.22
Routing:
- net BNO_RST: track 45.1 -> 0.00 mm
- net SDA2: track 0.00 -> 34.9 mm, vias 0 -> 3
- net SCL2: track 0.00 -> 33.5 mm, vias 0 -> 3
- net 3.3V: track 6.49 -> 31.3 mm
- net RX2: track 46.8 -> 42.6 mm, vias 2 -> 0
- net TX2: track 45.6 -> 44.3 mm, vias 2 -> 0
- net 3V3_SWITCH: track 111.3 -> 110.7 mm
- net N$73: track 30.6 -> 31.1 mm
