File: eagle/assets/layer4/layer4.sch (EAGLE design)
At the start: 45 parts, among them Y1 8MHz

Commit message: done with layer 4
Parts:
- renumbered BNO_RESET to COMPASS_RST
Changed lines of the file:
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@@
 <part name="GND5" library="SparkFun-PowerSymbols" deviceset="GND" device=""/>
 <part name="GND6" library="SparkFun-PowerSymbols" deviceset="GND" device=""/>
-<part name="BNO_RESET" library="MY-LIBRARY" library_urn="urn:adsk.eagle:library:11016882" deviceset="MOMENTARY_SWITCH_4X3" device="" package3d_urn="urn:adsk.eagle:package:11016890/3" value="MOMENTARY_SWITCH_4X3"/>
+<part name="COMPASS_RST" library="MY-LIBRARY" library_urn="urn:adsk.eagle:library:11016882" deviceset="MOMENTARY_SWITCH_4X3" device="" package3d_urn="urn:adsk.eagle:package:11016890/3" value="MOMENTARY_SWITCH_4X3"/>
 <part name="SUPPLY33" library="SparkFun-PowerSymbols" deviceset="3.3V" device=""/>
 <part name="3V3_PWR" library="SparkFun-Switches" library_urn="urn:adsk.eagle:library:11044690" deviceset="SWITCH-SPDT" device="-PTH-11.6X4.0MM-LOCK" package3d_urn="urn:adsk.eagle:package:11044812/2"/>
@@
 <attribute name="VALUE" x="193.04" y="88.646" size="1.778" layer="96" align="top-center"/>
 </instance>
-<instance part="BNO_RESET" gate="G$1" x="193.04" y="96.52" smashed="yes" rot="R90">
-<attribute name="NAME" x="200.66" y="97.536" size="1.778" layer="95" font="vector" rot="R180" align="bottom-center"/>
+<instance part="COMPASS_RST" gate="G$1" x="193.04" y="96.52" smashed="yes" rot="R90">
+<attribute name="NAME" x="200.66" y="97.536" size="1.778" layer="95" rot="R180" align="bottom-center"/>
 </instance>
 <instance part="SUPPLY33" gate="G$1" x="172.72" y="73.66" smashed="yes">
@@
 </segment>
 <segment>
-<pinref part="BNO_RESET" gate="G$1" pin="1"/>
+<pinref part="COMPASS_RST" gate="G$1" pin="1"/>
 <pinref part="GND6" gate="1" pin="GND"/>
 </segment>
@@
 <wire x1="180.34" y1="101.6" x2="193.04" y2="101.6" width="0.1524" layer="91"/>
 <label x="180.34" y="101.6" size="1.778" layer="95"/>
-<pinref part="BNO_RESET" gate="G$1" pin="2"/>
-</segment>
-</net>
+<pinref part="COMPASS_RST" gate="G$1" pin="2"/>
+</segment>
+</net>

Commit message: Edited Layer 4
Parts:
- removed COMPASS_RST: MOMENTARY_SWITCH_4X3, MY-LIBRARY:MOMENTARY_SWITCH_4X3
- added R6, R7: 4.7k, SparkFun-Resistors:4.7KOHM-0603-1/10W-1%
Connections:
- removed net BNO_RST: COMPASS.RESET, COMPASS_RST.2, STM32.PB0/ADC12_IN8/TIM3_CH3
- net 3.3V: now also R6.2, R7.2
- net GND: no longer COMPASS.I2C_SEL, COMPASS_RST.1
- net SCL2: now also R7.1, STM32.PB10/I2C2_SCL/USART3_TX
- net SDA2: now also R6.1, STM32.PB11/I2C2_SDA/USART3_RX
Changed lines of the file:
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@@
 <part name="3RD_LAYER" library="con-JST SH" library_urn="urn:adsk.eagle:library:16859530" deviceset="SM04B-SRSS" device="-TB" package3d_urn="urn:adsk.eagle:package:16859588/2"/>
 <part name="COMPASS" library="JH" library_urn="urn:adsk.eagle:library:6027132" deviceset="BNO055" device="" package3d_urn="urn:adsk.eagle:package:16833735/3"/>
-<part name="GND5" library="SparkFun-PowerSymbols" deviceset="GND" device=""/>
-<part name="GND6" library="SparkFun-PowerSymbols" deviceset="GND" device=""/>
-<part name="COMPASS_RST" library="MY-LIBRARY" library_urn="urn:adsk.eagle:library:11016882" deviceset="MOMENTARY_SWITCH_4X3" device="" package3d_urn="urn:adsk.eagle:package:11016890/3" value="MOMENTARY_SWITCH_4X3"/>
 <part name="SUPPLY33" library="SparkFun-PowerSymbols" deviceset="3.3V" device=""/>
 <part name="3V3_PWR" library="SparkFun-Switches" library_urn="urn:adsk.eagle:library:11044690" deviceset="SWITCH-SPDT" device="-PTH-11.6X4.0MM-LOCK" package3d_urn="urn:adsk.eagle:package:11044812/2"/>
+<part name="SUPPLY2" library="SparkFun-PowerSymbols" deviceset="3.3V" device=""/>
+<part name="SUPPLY3" library="SparkFun-PowerSymbols" deviceset="3.3V" device=""/>
+<part name="R6" library="SparkFun-Resistors" library_urn="urn:adsk.eagle:library:532" deviceset="4.7KOHM" device="-0603-1/10W-1%" package3d_urn="urn:adsk.eagle:package:39650/1" value="4.7k"/>
+<part name="R7" library="SparkFun-Resistors" library_urn="urn:adsk.eagle:library:532" deviceset="4.7KOHM" device="-0603-1/10W-1%" package3d_urn="urn:adsk.eagle:package:39650/1" value="4.7k"/>
+<part name="GND1" library="SparkFun-PowerSymbols" library_urn="urn:adsk.eagle:library:530" deviceset="GND" device=""/>
 </parts>
 <sheets>
@@
 <attribute name="NAME" x="162.56" y="119.888" size="1.27" layer="95"/>
 </instance>
-<instance part="GND5" gate="1" x="200.66" y="104.14" smashed="yes">
-<attribute name="VALUE" x="200.66" y="103.886" size="1.778" layer="96" align="top-center"/>
-</instance>
-<instance part="GND6" gate="1" x="193.04" y="88.9" smashed="yes">
-<attribute name="VALUE" x="193.04" y="88.646" size="1.778" layer="96" align="top-center"/>
-</instance>
-<instance part="COMPASS_RST" gate="G$1" x="193.04" y="96.52" smashed="yes" rot="R90">
-<attribute name="NAME" x="200.66" y="97.536" size="1.778" layer="95" rot="R180" align="bottom-center"/>
-</instance>
 <instance part="SUPPLY33" gate="G$1" x="172.72" y="73.66" smashed="yes">
 <attribute name="VALUE" x="172.72" y="76.454" size="1.778" layer="96" align="bottom-center"/>
@@
 <attribute name="NAME" x="175.768" y="69.85" size="1.778" layer="95" font="vector" rot="R270" align="bottom-center"/>
 <attribute name="VALUE" x="169.418" y="70.104" size="1.778" layer="96" font="vector" rot="R270" align="top-center"/>
+</instance>
+<instance part="SUPPLY2" gate="G$1" x="236.22" y="111.76" smashed="yes" rot="R270">
+<attribute name="VALUE" x="239.014" y="111.76" size="1.778" layer="96" rot="R270" align="bottom-center"/>
+</instance>
+<instance part="SUPPLY3" gate="G$1" x="236.22" y="99.06" smashed="yes" rot="R270">
+<attribute name="VALUE" x="239.014" y="99.06" size="1.778" layer="96" rot="R270" align="bottom-center"/>
+</instance>
+<instance part="R6" gate="G$1" x="228.6" y="111.76" smashed="yes">
+<attribute name="NAME" x="228.6" y="113.284" size="1.778" layer="95" font="vector" align="bottom-center"/>
+<attribute name="VALUE" x="228.6" y="110.236" size="1.778" layer="96" font="vector" align="top-center"/>
+</instance>
+<instance part="R7" gate="G$1" x="228.6" y="99.06" smashed="yes">
+<attribute name="NAME" x="228.6" y="100.584" size="1.778" layer="95" font="vector" align="bottom-center"/>
+<attribute name="VALUE" x="228.6" y="97.536" size="1.778" layer="96" font="vector" align="top-center"/>
+</instance>
+<instance part="GND1" gate="1" x="199.898" y="114.3" smashed="yes" rot="R90">
+<attribute name="VALUE" x="202.692" y="114.3" size="1.778" layer="96" rot="R270" align="top-center"/>
 </instance>
 </instances>
@@
 </segment>
 </net>
-<net name="GND" class="0">
-<segment>
-<pinref part="COMPASS" gate="G$1" pin="GND"/>
-<pinref part="GND5" gate="1" pin="GND"/>
-<wire x1="180.34" y1="114.3" x2="200.66" y2="114.3" width="0.1524" layer="91"/>
-<wire x1="200.66" y1="114.3" x2="200.66" y2="106.68" width="0.1524" layer="91"/>
-<pinref part="COMPASS" gate="G$1" pin="I2C_SEL"/>
-<wire x1="200.66" y1="106.68" x2="180.34" y2="106.68" width="0.1524" layer="91"/>
-<junction x="200.66" y="106.68"/>
-</segment>
-<segment>
-<pinref part="COMPASS_RST" gate="G$1" pin="1"/>
-<pinref part="GND6" gate="1" pin="GND"/>
-</segment>
-</net>
 <net name="3V3_SWITCH" class="0">
 <segment>
@@
 </segment>
 </net>
-<net name="BNO_RST" class="0">
-<segment>
-<pinref part="COMPASS" gate="G$1" pin="RESET"/>
-<wire x1="180.34" y1="101.6" x2="193.04" y2="101.6" width="0.1524" layer="91"/>
-<label x="180.34" y="101.6" size="1.778" layer="95"/>
-<pinref part="COMPASS_RST" gate="G$1" pin="2"/>
-</segment>
-</net>
 <net name="SDA2" class="0">
 <segment>
@@
 <label x="182.88" y="111.76" size="1.778" layer="95"/>
 </segment>
+<segment>
+<label x="223.52" y="106.68" size="1.778" layer="95" rot="R90"/>
+<wire x1="223.52" y1="115.57" x2="223.52" y2="111.76" width="0.1524" layer="91"/>
+<pinref part="R6" gate="G$1" pin="1"/>
+<wire x1="223.52" y1="111.76" x2="223.52" y2="106.68" width="0.1524" layer="91"/>
+<junction x="223.52" y="111.76"/>
+</segment>
 </net>
 <net name="SCL2" class="0">
@@
 <label x="182.88" y="109.22" size="1.778" layer="95"/>
 </segment>
+<segment>
+<label x="223.52" y="93.98" size="1.778" layer="95" rot="R90"/>
+<wire x1="223.52" y1="103.124" x2="223.52" y2="99.06" width="0.1524" layer="91"/>
+<pinref part="R7" gate="G$1" pin="1"/>
+<wire x1="223.52" y1="99.06" x2="223.52" y2="93.98" width="0.1524" layer="91"/>
+<junction x="223.52" y="99.06"/>
+</segment>
 </net>
 <net name="3.3V" class="0">
@@
 <pinref part="SUPPLY33" gate="G$1" pin="3.3V"/>
 <pinref part="3V3_PWR" gate="1" pin="P"/>
+</segment>
+<segment>
+<pinref part="SUPPLY2" gate="G$1" pin="3.3V"/>
+<wire x1="233.68" y1="111.76" x2="236.22" y2="111.76" width="0.1524" layer="91"/>
+<pinref part="R6" gate="G$1" pin="2"/>
+</segment>
+<segment>
+<pinref part="SUPPLY3" gate="G$1" pin="3.3V"/>
+<wire x1="233.68" y1="99.06" x2="236.22" y2="99.06" width="0.1524" layer="91"/>
+<pinref part="R7" gate="G$1" pin="2"/>
+</segment>
+</net>
+<net name="GND" class="0">
+<segment>
+<pinref part="COMPASS" gate="G$1" pin="GND"/>
+<wire x1="180.34" y1="114.3" x2="197.358" y2="114.3" width="0.1524" layer="91"/>
+<pinref part="GND1" gate="1" pin="GND"/>
 </segment>
 </net>
@@
 </segment>
 </net>
-<net name="BNO_RST" class="0">
-<segment>
-<pinref part="STM32" gate="G$1" pin="PB0/ADC12_IN8/TIM3_CH3"/>
-<wire x1="101.6" y1="78.74" x2="88.9" y2="78.74" width="0.1524" layer="91"/>
-<label x="88.9" y="78.74" size="1.778" layer="95"/>
-</segment>
-</net>
 <net name="L2C" class="0">
 <segment>
@@
 </segment>
 </net>
+<net name="SDA2" class="0">
+<segment>
+<pinref part="STM32" gate="G$1" pin="PB11/I2C2_SDA/USART3_RX"/>
+<wire x1="101.6" y1="68.58" x2="88.9" y2="68.58" width="0.1524" layer="91"/>
+<label x="88.9" y="68.58" size="1.778" layer="95"/>
+</segment>
+</net>
+<net name="SCL2" class="0">
+<segment>
+<pinref part="STM32" gate="G$1" pin="PB10/I2C2_SCL/USART3_TX"/>
+<wire x1="101.6" y1="71.12" x2="88.9" y2="71.12" width="0.1524" layer="91"/>
+<label x="88.9" y="71.12" size="1.778" layer="95"/>
+</segment>
+</net>
