File: eagle/assets/layer1/Layer 1.brd (EAGLE design)
At the start: 196 x 185.3 mm, 245 parts, among them M1C1 33nF, M1C2 680uF, M1C3 1.0uF, M1D1 RED, M1D2 BLUE, M1J1 XT30PB-F, M1Q1 AOD482, M1R1 1k, M1R10 1k, M1R11 10k, M1R12 4.7k, M1R2 1k, M1R3 3.3k, M1R4 3.3k, M1R5 1k, M1R6 1k, M1R7 1k, M1R8 10k, M1R9 10k, M2C1 33nF, M2C2 680uF, M2C3 1.0uF, M2D1 RED, M2D2 BLUE, M2J1 XT30PB-F, M2Q1 AOD482, M2R1 1k, M2R10 1k, M2R11 10k, M2R12 4.7k, M2R2 1k, M2R3 3.3k, M2R4 3.3k, M2R5 1k, M2R6 1k, M2R7 1k, M2R8 10k, M2R9 10k, M3C1 33nF, M3C2 680uF, M3C3 1.0uF, M3D1 RED, M3D2 BLUE, M3J1 XT30PB-F, M3Q1 AOD482, M3R1 1k, M3R10 1k, M3R11 10k, M3R12 4.7k, M3R2 1k, M3R3 3.3k, M3R4 3.3k, M3R5 1k, M3R6 1k, M3R7 1k, M3R8 10k, M3R9 10k, M4C1 33nF, M4C2 680uF, M4C3 1.0uF, M4D1 RED, M4D2 BLUE, M4J1 XT30PB-F, M4Q1 AOD482, M4R1 1k, M4R10 1k, M4R11 10k, M4R12 4.7k, M4R2 1k, M4R3 3.3k, M4R4 3.3k, M4R5 1k, M4R6 1k, M4R7 1k, M4R8 10k, M4R9 10k, Q37 AO3402, X2 SM06B-SRSS-TB, Y1 8MHz

Commit message: Depressed 🦅
Routing:
- net LS1: track 192.7 -> 192.1 mm

Commit message: Depressed 🦅 Layer 1
Parts:
- moved 1C4 4.65 mm to (-0.63, -59.2)
- moved 1C5 2.00 mm to (7.61, -59.8)
- moved LC3 0.08 mm to (-54.3, -34.0), turned to 145 degrees
Routing:
- net AGND: track 255.5 -> 259.2 mm
- net N$94: track 27.6 -> 30.4 mm
- net N$95: track 38.6 -> 41.3 mm
- net 3.3V: track 508.2 -> 510.6 mm
- net LS2: track 222.4 -> 220.6 mm
- net VCCA: track 563.8 -> 564.7 mm
- net V_BATT: track 221.8 -> 221.1 mm
- net M_SWITCH: track 326.9 -> 327.5 mm
- net LSWITCH: track 485.8 -> 486.3 mm
- net GND: track 36.3 -> 36.0 mm, vias 46 -> 47
Other:
- board text added: "V_BATT"

Commit message: Done layer 1
Routing:
- net AGND: track 259.2 -> 262.3 mm
- net LSIG2: track 112.6 -> 113.2 mm
Changed lines of the file:
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@@
 <drawing>
 <settings>
-<setting alwaysvectorfont="yes"/>
+<setting alwaysvectorfont="no"/>
 <setting verticaltext="up"/>
 </settings>
@@
 </layers>
 <board>
-<fusionsync huburn="a.YnVzaW5lc3M6Z21haWwxNDMxNzc3" projecturn="a.YnVzaW5lc3M6Z21haWwxNDMxNzc3IzIwMjIwMTE1NDg1NTYyMzgx" f3durn="urn:adsk.wipprod:dm.lineage:nDmFgUl6RZa3eTa8bgo8tA" pcbguid="" lastpulledtime="" lastsyncedchangeguid="" latestrevisionid="181ee6b0-77de-42b4-b011-61a22a925846" lastsyncedrevisionid="181ee6b0-77de-42b4-b011-61a22a925846" lastboardhashguid="7a93af17-8a7a-dd58-67c8-bf5800a77ba0" lastpushedtime="2022-02-25T06:11:01Z" linktopcb3d="false"/>
+<fusionsync huburn="a.YnVzaW5lc3M6Z21haWwxNDMxNzc3" projecturn="a.YnVzaW5lc3M6Z21haWwxNDMxNzc3IzIwMjIwMTE1NDg1NTYyMzgx" f3durn="urn:adsk.wipprod:dm.lineage:nDmFgUl6RZa3eTa8bgo8tA" pcbguid="" lastpulledtime="" lastsyncedchangeguid="" latestrevisionid="73b57eb6-1d62-4e71-a84d-98288279c7f9" lastsyncedrevisionid="73b57eb6-1d62-4e71-a84d-98288279c7f9" lastboardhashguid="4a9ab027-583b-8016-6be8-8ccc89b62292" lastpushedtime="2022-02-25T06:33:48Z" linktopcb3d="true"/>
 <plain>
 <text x="-55.5" y="-9.2" size="0.6096" layer="25" rot="R90">3.3V</text>
@@
 <via x="-28.64358125" y="-16.28648125" extent="1-16" drill="0.508"/>
 <via x="-37.26941875" y="-29.220159375" extent="1-16" drill="0.508"/>
-<via x="-39.283640625" y="-43.266359375" extent="1-16" drill="0.508"/>
 <via x="42.097959375" y="-38.287959375" extent="1-16" drill="0.508"/>
 <via x="27.97301875" y="-38.6842" extent="1-16" drill="0.508"/>
@@
 <via x="27.675" y="-13.245" extent="1-16" drill="0.508"/>
 <via x="-27" y="-5" extent="1-16" drill="0.508"/>
+<via x="-0.84" y="-20.675" extent="1-16" drill="0.508"/>
 </signal>
 <signal name="N$2">
@@
 <wire x1="-14.375" y1="-45.575" x2="-14.73035" y2="-45.93035" width="0.254" layer="1"/>
 <via x="-17.254953125" y="-45.9342625" extent="1-16" drill="0.508"/>
-<wire x1="-18.29941875" y1="-36.466978125" x2="-17.263475" y2="-35.431034375" width="0.254" layer="16"/>
-<wire x1="-17.263475" y1="-35.431034375" x2="-8.592340625" y2="-35.431034375" width="0.254" layer="16"/>
-<wire x1="-8.592340625" y1="-35.431034375" x2="-6.10725" y2="-32.94594375" width="0.254" layer="16"/>
-<wire x1="-18.29941875" y1="-36.466978125" x2="-18.29941875" y2="-44.889796875" width="0.254" layer="16"/>
+<wire x1="-18.29941875" y1="-35.481978125" x2="-15.763384375" y2="-32.94594375" width="0.254" layer="16"/>
+<wire x1="-18.29941875" y1="-35.481978125" x2="-18.29941875" y2="-44.889796875" width="0.254" layer="16"/>
 <wire x1="-17.254953125" y1="-45.9342625" x2="-18.29941875" y2="-44.889796875" width="0.254" layer="16"/>
 <wire x1="20.709740625" y1="-32.94594375" x2="21.8992375" y2="-31.756446875" width="0.254" layer="16"/>
@@
 <wire x1="21.8992375" y1="-31.756446875" x2="21.8992375" y2="-11.164440625" width="0.254" layer="16"/>
 <wire x1="21.8992375" y1="-11.164440625" x2="21.95880625" y2="-11.104871875" width="0.254" layer="16"/>
-<wire x1="-6.10725" y1="-32.94594375" x2="20.709740625" y2="-32.94594375" width="0.254" layer="16"/>
+<wire x1="-15.763384375" y1="-32.94594375" x2="20.709740625" y2="-32.94594375" width="0.254" layer="16"/>
 <wire x1="11.163821875" y1="3.541796875" x2="11.163821875" y2="4.694903125" width="0.254" layer="16"/>
 <wire x1="11.163821875" y1="4.694903125" x2="11.384459375" y2="4.915540625" width="0.254" layer="16"/>
@@
 <wire x1="-17.0359125" y1="-48.8061" x2="-18.087340625" y2="-48.8061" width="0.254" layer="1"/>
 <via x="-18.087340625" y="-48.8061" extent="1-16" drill="0.508"/>
-<via x="-29.792634375" y="-34.2452375" extent="1-16" drill="0.508"/>
-<wire x1="-27.369384375" y1="-48.817103125" x2="-29.792634375" y2="-46.393853125" width="0.254" layer="16"/>
-<wire x1="-29.792634375" y1="-46.393853125" x2="-29.792634375" y2="-34.2452375" width="0.254" layer="16"/>
+<via x="-39.367634375" y="-32.0052375" extent="1-16" drill="0.508"/>
+<wire x1="-32.414384375" y1="-48.817103125" x2="-39.367634375" y2="-41.863853125" width="0.254" layer="16"/>
+<wire x1="-39.367634375" y1="-41.863853125" x2="-39.367634375" y2="-32.0052375" width="0.254" layer="16"/>
 <wire x1="-18.087340625" y1="-48.8061" x2="-18.09834375" y2="-48.817103125" width="0.254" layer="16"/>
-<wire x1="-18.09834375" y1="-48.817103125" x2="-27.369384375" y2="-48.817103125" width="0.254" layer="16"/>
-<wire x1="-29.792634375" y1="-34.2452375" x2="-39.14723125" y2="-24.890640625" width="0.254" layer="1"/>
+<wire x1="-18.09834375" y1="-48.817103125" x2="-32.414384375" y2="-48.817103125" width="0.254" layer="16"/>
+<wire x1="-39.367634375" y1="-32.0052375" x2="-39.14723125" y2="-31.784834375" width="0.254" layer="1"/>
 <wire x1="-39.14723125" y1="2.40265625" x2="-39.0290625" y2="2.520825" width="0.254" layer="1"/>
-<wire x1="-39.14723125" y1="2.40265625" x2="-39.14723125" y2="-24.890640625" width="0.254" layer="1"/>
+<wire x1="-39.14723125" y1="2.40265625" x2="-39.14723125" y2="-31.784834375" width="0.254" layer="1"/>
 <wire x1="-3.837925" y1="2.274190625" x2="-2.337925" y2="2.274190625" width="0.254" layer="16"/>
 <wire x1="12.26326875" y1="-47.17976875" x2="12.242828125" y2="-47.200209375" width="0.254" layer="16"/>
@@
 <wire x1="29.81198125" y1="-26.293075" x2="29.81198125" y2="-34.50478125" width="0.254" layer="16"/>
 <wire x1="29.81198125" y1="-34.50478125" x2="29.1631625" y2="-35.1536" width="0.254" layer="16"/>
-<wire x1="-9.049865625" y1="-36.535140625" x2="-15.369253125" y2="-36.535140625" width="0.254" layer="16"/>
+<wire x1="-15.354865625" y1="-36.535140625" x2="-15.369253125" y2="-36.535140625" width="0.254" layer="16"/>
 <via x="-32.06365" y="-33.169059375" extent="1-16" drill="0.508"/>
-<wire x1="29.1631625" y1="-35.1536" x2="-7.668325" y2="-35.1536" width="0.254" layer="16"/>
-<wire x1="-7.668325" y1="-35.1536" x2="-9.049865625" y2="-36.535140625" width="0.254" layer="16"/>
+<wire x1="29.1631625" y1="-35.1536" x2="-13.973325" y2="-35.1536" width="0.254" layer="16"/>
+<wire x1="-13.973325" y1="-35.1536" x2="-15.354865625" y2="-36.535140625" width="0.254" layer="16"/>
 <via x="-15.369253125" y="-36.535140625" extent="1-16" drill="0.508"/>
 <wire x1="-28.078953125" y1="-37.15375625" x2="-15.98786875" y2="-37.15375625" width="0.254" layer="1"/>
@@
 <wire x1="0.00798125" y1="-49.803890625" x2="-0.00794375" y2="-49.819815625" width="0.254" layer="1"/>
 </signal>
-<signal name="N$109">
-<via x="-4" y="-77.42443125" extent="1-16" drill="3.2" diameter="7"/>
-</signal>
-<signal name="N$110">
-<via x="4" y="-77.42443125" extent="1-16" drill="3.2" diameter="7"/>
-</signal>
-<signal name="N$111">
-<via x="4" y="-69.42443125" extent="1-16" drill="3.2" diameter="7"/>
-</signal>
-<signal name="N$112">
-<via x="-4" y="-69.42443125" extent="1-16" drill="3.2" diameter="7"/>
-</signal>
 </signals>

Commit message: Finished
Parts:
- moved LDR 4.05 mm to (40.0, 76.0), turned to 270 degrees
- moved LG_R2 3.09 mm to (40.8, 71.4), turned to 180 degrees
- moved LED 1.60 mm to (-40.0, 76.0)
- moved 2C4 1.20 mm to (4.05, 54.7), turned to 180 degrees
- moved 2R4 1.15 mm to (4.05, 53.1), turned to 0 degrees
- moved LC1 1.00 mm to (-40.5, 69.9)
Routing:
- net VCCA: track 564.7 -> 569.5 mm
- net LG_SIG: track 101.4 -> 99.3 mm
- net AGND: track 262.3 -> 261.0 mm
- net LSWITCH: track 486.3 -> 487.5 mm

Commit message: fuck i do eagle again
Parts:
- moved X2 95.8 mm to (7.54, -68.9), turned to 180 degrees
- moved 1C10 7.61 mm to (43.5, -9.74), turned to 180 degrees
- moved 1L1 4.35 mm to (17.5, -59.1), turned to 180 degrees
- moved 1C6 3.76 mm to (48.0, -10.6), turned to 270 degrees
- moved R1 3.52 mm to (-88.5, 13.5), turned to 180 degrees
- moved 1C2 2.81 mm to (33.7, -68.0), turned to 180 degrees
- moved 2C2 2.60 mm to (-24.1, -46.8)
- moved 1D1 2.00 mm to (26.3, -61.4)
- moved C6 1.92 mm to (7.33, 6.69)
- moved Y1 1.90 mm to (10.00, 9.42)
- moved LC5 1.80 mm to (25.5, -60.3)
- moved R2 1.68 mm to (-84.2, 7.36), turned to 180 degrees
- moved 1C1 1.68 mm to (36.3, -71.4)
- moved RST 1.40 mm to (-85.0, 11.2)
- moved C7 1.35 mm to (10.8, 6.77)
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Routing:
- net SWDIO: track 94.0 -> 165.2 mm, vias 5 -> 1
- net RX1: track 126.8 -> 158.9 mm, vias 3 -> 4
- net TX1: track 131.8 -> 155.5 mm, vias 3 -> 4
- net SWCLK: track 132.1 -> 154.1 mm, vias 7 -> 5
- net V_BATT: track 221.1 -> 241.3 mm, vias 10 -> 11
- net 3.3V: track 510.6 -> 529.9 mm
- net N$2: track 28.8 -> 20.7 mm
- net VCCA: track 569.5 -> 575.6 mm
- net N$98: track 67.1 -> 71.4 mm
- net GND: track 36.0 -> 40.2 mm, vias 47 -> 28
- net RESET: track 107.4 -> 105.0 mm
- net N$96: track 52.0 -> 54.3 mm
- net LS2: track 220.6 -> 222.7 mm
- net N$97: track 58.9 -> 60.7 mm
- net LS1: track 192.1 -> 190.4 mm
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
Commit message: fuck i do eagle again
Parts:
- moved LC5 0.71 mm to (25.3, -61.0)
Routing:
- net LSWITCH: track 488.6 -> 489.3 mm
- net N$97: track 60.7 -> 60.1 mm
Changed lines of the file:
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@@
 </layers>
 <board>
-<fusionsync huburn="a.YnVzaW5lc3M6Z21haWwxNDMxNzc3" projecturn="a.YnVzaW5lc3M6Z21haWwxNDMxNzc3IzIwMjIwMTE1NDg1NTYyMzgx" f3durn="urn:adsk.wipprod:dm.lineage:nDmFgUl6RZa3eTa8bgo8tA" pcbguid="" lastpulledtime="" lastsyncedchangeguid="" latestrevisionid="d4c49dbf-dcfd-4069-becc-f1496cad887c" lastsyncedrevisionid="d4c49dbf-dcfd-4069-becc-f1496cad887c" lastboardhashguid="eafd83db-46f7-4b79-3f1a-3e0a5c6dd9f4" lastpushedtime="2022-02-26T14:22:50Z" linktopcb3d="true"/>
+<fusionsync huburn="a.YnVzaW5lc3M6Z21haWwxNDMxNzc3" projecturn="a.YnVzaW5lc3M6Z21haWwxNDMxNzc3IzIwMjIwMTE1NDg1NTYyMzgx" f3durn="urn:adsk.wipprod:dm.lineage:nDmFgUl6RZa3eTa8bgo8tA" pcbguid="" lastpulledtime="" lastsyncedchangeguid="" latestrevisionid="e7c7bbc5-9887-4801-a9f6-1a7a9b546ab0" lastsyncedrevisionid="e7c7bbc5-9887-4801-a9f6-1a7a9b546ab0" lastboardhashguid="cb09ae10-52a2-cf80-74c1-46140a957af2" lastpushedtime="2022-02-26T14:38:46Z" linktopcb3d="true"/>
 <plain>
 <text x="-55.5" y="-9.2" size="0.6096" layer="25" rot="R90">3.3V</text>
@@
 <attribute name="VALUE" x="-24.1636625" y="-61.9407375" size="0.7112" layer="27" font="vector" ratio="18" rot="R225" align="top-center"/>
 </element>
-<element name="LC5" library="JH" library_urn="urn:adsk.eagle:library:6027132" package="C0603" package3d_urn="urn:adsk.eagle:package:15441226/3" value="1uF" x="25.5" y="-60.3" smashed="yes" rot="MR0">
-<attribute name="VALUE" x="25.5" y="-61.062" size="0.7112" layer="28" font="vector" ratio="18" rot="MR0" align="top-center"/>
+<element name="LC5" library="JH" library_urn="urn:adsk.eagle:library:6027132" package="C0603" package3d_urn="urn:adsk.eagle:package:15441226/3" value="1uF" x="25.34" y="-60.995" smashed="yes" rot="MR0">
+<attribute name="VALUE" x="25.34" y="-61.757" size="0.7112" layer="28" font="vector" ratio="18" rot="MR0" align="top-center"/>
 </element>
 <element name="LC6" library="JH" library_urn="urn:adsk.eagle:library:6027132" package="C0603" package3d_urn="urn:adsk.eagle:package:15441226/3" value="1uF" x="54.3" y="-34" smashed="yes" rot="MR90">
@@
 <wire x1="54.3" y1="-34.85" x2="52.441109375" y2="-36.708890625" width="0.254" layer="16"/>
 <wire x1="52.441109375" y1="-36.708890625" x2="52.42573125" y2="-36.708890625" width="0.254" layer="16"/>
-<wire x1="26.35" y1="-60.3" x2="26.34999375" y2="-58.701271875" width="0.254" layer="16"/>
-<wire x1="26.34999375" y1="-58.701271875" x2="27.04756875" y2="-58.003696875" width="0.254" layer="16"/>
+<wire x1="26.19" y1="-60.995" x2="26.18999375" y2="-58.861271875" width="0.254" layer="16"/>
+<wire x1="26.18999375" y1="-58.861271875" x2="27.04756875" y2="-58.003696875" width="0.254" layer="16"/>
 <wire x1="-52.42573125" y1="-36.708890625" x2="-52.774928125" y2="-36.708890625" width="0.254" layer="16"/>
 <wire x1="-52.774928125" y1="-36.708890625" x2="-54.97128125" y2="-34.5125375" width="0.254" layer="16"/>
@@
 <contactref element="Q30" pad="E"/>
 <contactref element="MUX_L2" pad="7"/>
-<wire x1="21.632778125" y1="-59.43555625" x2="22.76029375" y2="-59.43555625" width="0.254" layer="16"/>
 <wire x1="-11.13488125" y1="-43.93101875" x2="-11.13488125" y2="-50.498615625" width="0.254" layer="1"/>
 <wire x1="-14.373665625" y1="-41.676334375" x2="-14.375" y2="-41.675" width="0.254" layer="1"/>
 <wire x1="-11.13488125" y1="-43.93101875" x2="-13.389565625" y2="-41.676334375" width="0.254" layer="1"/>
 <wire x1="-13.389565625" y1="-41.676334375" x2="-14.373665625" y2="-41.676334375" width="0.254" layer="1"/>
-<wire x1="23.034515625" y1="-59.161334375" x2="23.034515625" y2="-55.034515625" width="0.254" layer="1"/>
-<wire x1="23.034515625" y1="-55.034515625" x2="22" y2="-54" width="0.254" layer="1"/>
+<wire x1="23.049515625" y1="-55.049515625" x2="22" y2="-54" width="0.254" layer="1"/>
 <wire x1="22" y1="-54" x2="8.25" y2="-54" width="0.254" layer="1"/>
 <wire x1="8.25" y1="-54" x2="5.95" y2="-56.3" width="0.254" layer="1"/>
@@
 <via x="-1.786303125" y="-56.3" extent="1-16" drill="0.508"/>
 <wire x1="-11.13488125" y1="-50.498615625" x2="-5.333496875" y2="-56.3" width="0.254" layer="1"/>
-<wire x1="22.76029375" y1="-59.43555625" x2="23.034515625" y2="-59.161334375" width="0.254" layer="16"/>
-<via x="23.034515625" y="-59.161334375" extent="1-16" drill="0.508"/>
+<wire x1="23.049515625" y1="-55.049515625" x2="23.049515625" y2="-59.205484375" width="0.254" layer="1"/>
+<wire x1="21.632778125" y1="-59.43555625" x2="22.81944375" y2="-59.43555625" width="0.254" layer="16"/>
+<wire x1="22.81944375" y1="-59.43555625" x2="23.049515625" y2="-59.205484375" width="0.254" layer="16"/>
+<via x="23.049515625" y="-59.205484375" extent="1-16" drill="0.508"/>
 </signal>
 <signal name="N$97">
@@
 <wire x1="31.625" y1="-54.776103125" x2="31.625" y2="-55.022021875" width="0.254" layer="16"/>
 <wire x1="31.625" y1="-55.022021875" x2="30.0355" y2="-56.611521875" width="0.254" layer="16"/>
-<wire x1="16.6596375" y1="-55.35955" x2="19.76140625" y2="-52.25778125" width="0.254" layer="16"/>
+<wire x1="19.05640625" y1="-52.96278125" x2="16.6596375" y2="-55.35955" width="0.254" layer="16"/>
 <wire x1="-2.811475" y1="-55.35955" x2="-2.822496875" y2="-55.348528125" width="0.254" layer="16"/>
 <via x="-2.822496875" y="-55.348528125" extent="1-16" drill="0.508"/>
@@
 <wire x1="16.6596375" y1="-55.35955" x2="-2.811475" y2="-55.35955" width="0.254" layer="16"/>
 <wire x1="-5.56655" y1="-55.348528125" x2="-10.62188125" y2="-50.293196875" width="0.254" layer="1"/>
-<wire x1="19.76140625" y1="-52.25778125" x2="27.25778125" y2="-52.25778125" width="0.254" layer="16"/>
-<wire x1="27.25778125" y1="-52.25778125" x2="28" y2="-53" width="0.254" layer="16"/>
+<wire x1="19.05640625" y1="-52.96278125" x2="27.96278125" y2="-52.96278125" width="0.254" layer="16"/>
+<wire x1="27.96278125" y1="-52.96278125" x2="28" y2="-53" width="0.254" layer="16"/>
 <via x="28" y="-53" extent="1-16" drill="0.508"/>
-<wire x1="28" y1="-53" x2="30.0355" y2="-55.0355" width="0.254" layer="1"/>
-<wire x1="30.0355" y1="-55.0355" x2="30.0355" y2="-56.611521875" width="0.254" layer="1"/>
+<wire x1="28" y1="-53" x2="27.9955" y2="-53.0045" width="0.254" layer="1"/>
+<wire x1="27.9955" y1="-53.0045" x2="27.9955" y2="-54.571521875" width="0.254" layer="1"/>
+<wire x1="27.9955" y1="-54.571521875" x2="30.0355" y2="-56.611521875" width="0.254" layer="1"/>
 <via x="30.0355" y="-56.611521875" extent="1-16" drill="0.508"/>
 </signal>
@@
 <wire x1="-14.375" y1="-40.375" x2="-14.365996875" y2="-40.365996875" width="0.254" layer="1"/>
 <wire x1="-13.263053125" y1="-40.365996875" x2="-14.365996875" y2="-40.365996875" width="0.254" layer="1"/>
-<wire x1="16.2648125" y1="-54.349409375" x2="19.423903125" y2="-51.19031875" width="0.254" layer="16"/>
+<wire x1="16.2648125" y1="-54.349409375" x2="19.373903125" y2="-51.24031875" width="0.254" layer="16"/>
 <wire x1="-5.849128125" y1="-54.347528125" x2="-10.10888125" y2="-50.087775" width="0.254" layer="1"/>
 <via x="28.755459375" y="-51.255459375" extent="1-16" drill="0.508"/>
@@
 <wire x1="38.55290625" y1="-50.55571875" x2="40.656315625" y2="-48.452309375" width="0.254" layer="16"/>
 <wire x1="38.55290625" y1="-52.438978125" x2="38.55290625" y2="-50.55571875" width="0.254" layer="16"/>
-<wire x1="28.755459375" y1="-51.255459375" x2="28.69031875" y2="-51.19031875" width="0.254" layer="16"/>
-<wire x1="28.69031875" y1="-51.19031875" x2="19.423903125" y2="-51.19031875" width="0.254" layer="16"/>
+<wire x1="28.755459375" y1="-51.255459375" x2="28.74031875" y2="-51.24031875" width="0.254" layer="16"/>
+<wire x1="28.74031875" y1="-51.24031875" x2="19.373903125" y2="-51.24031875" width="0.254" layer="16"/>
 </signal>
 <signal name="N$99">
@@
 <wire x1="11.243721875" y1="-63.7663" x2="19.224603125" y2="-63.7663" width="0.254" layer="16"/>
 <wire x1="19.224603125" y1="-63.7663" x2="22.14580625" y2="-60.845096875" width="0.254" layer="16"/>
-<wire x1="27.3375875" y1="-62.11255625" x2="23.413265625" y2="-62.11255625" width="0.254" layer="16"/>
-<wire x1="22.14580625" y1="-60.845096875" x2="23.413265625" y2="-62.11255625" width="0.254" layer="16"/>
+<wire x1="26.9725875" y1="-62.47755625" x2="23.778265625" y2="-62.47755625" width="0.254" layer="16"/>
+<wire x1="22.14580625" y1="-60.845096875" x2="23.778265625" y2="-62.47755625" width="0.254" layer="16"/>
 <wire x1="32.375" y1="-57.07514375" x2="32.375" y2="-56.07514375" width="0.254" layer="16"/>
-<wire x1="32.375" y1="-57.07514375" x2="27.3375875" y2="-62.11255625" width="0.254" layer="16"/>
+<wire x1="32.375" y1="-57.07514375" x2="26.9725875" y2="-62.47755625" width="0.254" layer="16"/>
 <wire x1="32.375" y1="-56.07514375" x2="32.975" y2="-56.67514375" width="0.254" layer="16"/>
 <wire x1="35.8307875" y1="-56.67514375" x2="32.975" y2="-56.67514375" width="0.254" layer="16"/>
