File: eagle/assets/layer1/Layer 1.brd (EAGLE design)
At the start: 196 x 185.3 mm, 245 parts, among them M1C1 33nF, M1C2 680uF, M1C3 1.0uF, M1D1 RED, M1D2 BLUE, M1J1 XT30PB-F, M1Q1 AOD482, M1R1 1k, M1R10 1k, M1R11 10k, M1R12 4.7k, M1R2 1k, M1R3 3.3k, M1R4 3.3k, M1R5 1k, M1R6 1k, M1R7 1k, M1R8 10k, M1R9 10k, M2C1 33nF, M2C2 680uF, M2C3 1.0uF, M2D1 RED, M2D2 BLUE, M2J1 XT30PB-F, M2Q1 AOD482, M2R1 1k, M2R10 1k, M2R11 10k, M2R12 4.7k, M2R2 1k, M2R3 3.3k, M2R4 3.3k, M2R5 1k, M2R6 1k, M2R7 1k, M2R8 10k, M2R9 10k, M3C1 33nF, M3C2 680uF, M3C3 1.0uF, M3D1 RED, M3D2 BLUE, M3J1 XT30PB-F, M3Q1 AOD482, M3R1 1k, M3R10 1k, M3R11 10k, M3R12 4.7k, M3R2 1k, M3R3 3.3k, M3R4 3.3k, M3R5 1k, M3R6 1k, M3R7 1k, M3R8 10k, M3R9 10k, M4C1 33nF, M4C2 680uF, M4C3 1.0uF, M4D1 RED, M4D2 BLUE, M4J1 XT30PB-F, M4Q1 AOD482, M4R1 1k, M4R10 1k, M4R11 10k, M4R12 4.7k, M4R2 1k, M4R3 3.3k, M4R4 3.3k, M4R5 1k, M4R6 1k, M4R7 1k, M4R8 10k, M4R9 10k, Q37 AO3402, X2 SM06B-SRSS-TB, Y1 8MHz

Commit message: fuck i do eagle again
Parts:
- moved LR1 40.2 mm to (-46.3, 33.6), turned to 125 degrees
- moved R9 0.23 mm to (58.2, 4.33)
Routing:
- net N$69: track 421.7 -> 423.2 mm
Changed lines of the file:
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@@
 </layers>
 <board>
-<fusionsync huburn="a.YnVzaW5lc3M6Z21haWwxNDMxNzc3" projecturn="a.YnVzaW5lc3M6Z21haWwxNDMxNzc3IzIwMjIwMTE1NDg1NTYyMzgx" f3durn="urn:adsk.wipprod:dm.lineage:nDmFgUl6RZa3eTa8bgo8tA" pcbguid="" lastpulledtime="" lastsyncedchangeguid="" latestrevisionid="e7c7bbc5-9887-4801-a9f6-1a7a9b546ab0" lastsyncedrevisionid="e7c7bbc5-9887-4801-a9f6-1a7a9b546ab0" lastboardhashguid="cb09ae10-52a2-cf80-74c1-46140a957af2" lastpushedtime="2022-02-26T14:38:46Z" linktopcb3d="true"/>
+<fusionsync huburn="a.YnVzaW5lc3M6Z21haWwxNDMxNzc3" projecturn="a.YnVzaW5lc3M6Z21haWwxNDMxNzc3IzIwMjIwMTE1NDg1NTYyMzgx" f3durn="urn:adsk.wipprod:dm.lineage:nDmFgUl6RZa3eTa8bgo8tA" pcbguid="" lastpulledtime="" lastsyncedchangeguid="" latestrevisionid="41e871a6-fb33-4710-92c0-60d424b2d48b" lastsyncedrevisionid="41e871a6-fb33-4710-92c0-60d424b2d48b" lastboardhashguid="2f259927-8036-c267-1644-e3a054a40ded" lastpushedtime="2022-02-26T14:42:48Z" linktopcb3d="true"/>
 <plain>
 <text x="-55.5" y="-9.2" size="0.6096" layer="25" rot="R90">3.3V</text>
@@
 <attribute name="NAME" x="2.704496875" y="52.999996875" size="0.6604" layer="26" ratio="16" rot="MR270" align="center"/>
 </element>
-<element name="LR1" library="JH" library_urn="urn:adsk.eagle:library:6027132" package="R0603" package3d_urn="urn:adsk.eagle:package:15441228/3" value="47" x="-57.8" y="-5" smashed="yes" rot="MR180">
-<attribute name="NAME" x="-57.8" y="-5.762" size="0.7112" layer="26" font="vector" ratio="18" rot="MR180" align="bottom-center"/>
-<attribute name="VALUE" x="-57.8" y="-4.238" size="0.7112" layer="28" font="vector" ratio="18" rot="MR180" align="top-center"/>
+<element name="LR1" library="JH" library_urn="urn:adsk.eagle:library:6027132" package="R0603" package3d_urn="urn:adsk.eagle:package:15441228/3" value="47" x="-46.33" y="33.56" smashed="yes" rot="MR125">
+<attribute name="NAME" x="-45.705809375" y="33.1229375" size="0.7112" layer="26" font="vector" ratio="18" rot="MR125" align="bottom-center"/>
+<attribute name="VALUE" x="-46.95419375" y="33.997065625" size="0.7112" layer="28" font="vector" ratio="18" rot="MR125" align="top-center"/>
 </element>
 <element name="LIGHT_SWITCH" library="SparkFun-Switches" library_urn="urn:adsk.eagle:library:11044690" package="SWITCH_SPDT_PTH_11.6X4.0MM_LOCK" package3d_urn="urn:adsk.eagle:package:11044812/2" value="" x="-85.950984375" y="-11.864178125" smashed="yes">
@@
 <attribute name="VALUE" x="53.5400375" y="7.938484375" size="0.7112" layer="28" font="vector" ratio="18" rot="MR180" align="top-center"/>
 </element>
-<element name="R9" library="JH" library_urn="urn:adsk.eagle:library:6027132" package="R0603" package3d_urn="urn:adsk.eagle:package:15441228/3" value="4.7k" x="57.971321875" y="4.330571875" smashed="yes" rot="MR270">
-<attribute name="VALUE" x="58.733321875" y="4.330571875" size="0.7112" layer="28" font="vector" ratio="18" rot="MR270" align="top-center"/>
+<element name="R9" library="JH" library_urn="urn:adsk.eagle:library:6027132" package="R0603" package3d_urn="urn:adsk.eagle:package:15441228/3" value="4.7k" x="58.2" y="4.330571875" smashed="yes" rot="MR270">
+<attribute name="VALUE" x="58.962" y="4.330571875" size="0.7112" layer="28" font="vector" ratio="18" rot="MR270" align="top-center"/>
 </element>
 <element name="RST" library="MY-LIBRARY" library_urn="urn:adsk.eagle:library:11016882" package="MOMENTARY_SWITCH_4X3" package3d_urn="urn:adsk.eagle:package:11016890/3" value="MOMENTARY_SWITCH_4X3" x="-85" y="11.248165625" smashed="yes" rot="R90">
@@
 <wire x1="60.767878125" y1="-5.3165" x2="60.6457125" y2="-5.194334375" width="0.254" layer="16"/>
 <wire x1="60.6457125" y1="-5.194334375" x2="60.6457125" y2="5.438665625" width="0.254" layer="16"/>
-<wire x1="-60.767878125" y1="-5.3165" x2="-58.9665" y2="-5.3165" width="0.254" layer="16"/>
-<wire x1="-58.9665" y1="-5.3165" x2="-58.65" y2="-5" width="0.254" layer="16"/>
 <wire x1="-58.921478125" y1="15.787959375" x2="-58.921478125" y2="18.6091375" width="0.254" layer="16"/>
 <wire x1="-58.921478125" y1="18.6091375" x2="-59.103259375" y2="18.79091875" width="0.254" layer="16"/>
@@
 <wire x1="14.4" y1="51.13524375" x2="14.2886375" y2="51.02388125" width="0.254" layer="16"/>
 <wire x1="7.162903125" y1="-58.921475" x2="15.7879625" y2="-58.921475" width="0.254" layer="16"/>
+<wire x1="-49.968278125" y1="34.9881625" x2="-46.817540625" y2="32.86371875" width="0.254" layer="16"/>
 </signal>
 <signal name="LSIG1">
@@
 <contactref element="R9" pad="1"/>
 <contactref element="Q37" pad="1"/>
-<wire x1="57.971321875" y1="5.180571875" x2="56.571321875" y2="5.180571875" width="0.508" layer="16"/>
+<wire x1="58.2" y1="5.180571875" x2="56.571321875" y2="5.180571875" width="0.508" layer="16"/>
 <wire x1="56.571321875" y1="5.180571875" x2="56.471321875" y2="5.280571875" width="0.508" layer="16"/>
 </signal>
@@
 <contactref element="Q37" pad="2"/>
 <contactref element="J1" pad="1"/>
-<wire x1="57.971321875" y1="3.480571875" x2="57.871321875" y2="3.380571875" width="0.508" layer="16"/>
+<wire x1="58.2" y1="3.480571875" x2="57.871321875" y2="3.380571875" width="0.508" layer="16"/>
 <wire x1="57.871321875" y1="3.380571875" x2="56.471321875" y2="3.380571875" width="0.508" layer="16"/>
 <wire x1="56.471321875" y1="3.380571875" x2="53.45189375" y2="0.36114375" width="0.508" layer="16"/>

Commit message: final
Routing:
- net GND: vias 28 -> 29
Other:
- outline, holes or cut-outs redrawn
