File: elec/eagle/assets/layer3/layer3.brd (EAGLE design)
At the start: 196 x 158 mm, 84 parts, among them Q2 AO3402, X1 SM06B-SRSS-TB, Y1 8MHz

Commit message: layer 4 pcb
Parts:
- removed BNO055: (no value), SparkFun-Connectors:1X08_LOCK
- removed R10, R11: 4.7k, SparkFun-Resistors:0603
Connections:
- removed net MISO: TEENSY4.D12, U$8.12
- removed net MOSI: TEENSY4.D11, U$8.11
- removed net SCK: TEENSY4.D13/LED, U$8.13
- removed net SCL0_TEE: TEENSY4.D17/A3, U$8.15
- removed net SDA0_TEE: TEENSY4.D16/A2, U$8.16
- removed net SS: TEENSY4.D10, U$8.14
- new net RX_CAM: TEENSY4.D17/A3, U$8.16
- new net TX_CAM: TEENSY4.D16/A2, U$8.15
- net 3.3V: no longer R10.2, R11.2
- net 3V3_SWITCH: no longer BNO055.8
- net BL_DIR: now also TEENSY4.D11; no longer TEENSY4.D26
- net BR_DIR: now also TEENSY4.D6; no longer TEENSY4.D27
- net ESC_LV: now also TEENSY4.D9; no longer TEENSY4.D33
- net FL_DIR: now also TEENSY4.D12; no longer TEENSY4.D24
- net FR_DIR: now also TEENSY4.D13/LED; no longer TEENSY4.D25
- net GND: no longer BNO055.7
- net RX_BT: now also TEENSY4.D14/A0; no longer TEENSY4.D29
- net SCL1: no longer BNO055.5, R11.1
- net SDA1: no longer BNO055.6, R10.1
- net SERVO_LV: now also TEENSY4.D10; no longer TEENSY4.D30
- net TX_BT: now also TEENSY4.D15/A1; no longer TEENSY4.D28
Routing:
- net SDA1: track 102.4 -> 0.00 mm, vias 7 -> 0
- net SCL1: track 98.0 -> 0.00 mm, vias 7 -> 0
- net SCK: track 83.1 -> 0.00 mm, vias 3 -> 0
- net SDA0_TEE: track 82.7 -> 0.00 mm, vias 2 -> 0
- net SCL0_TEE: track 75.7 -> 0.00 mm
- net SS: track 72.0 -> 0.00 mm, vias 2 -> 0
- net TX_CAM: track 0.00 -> 71.6 mm, vias 0 -> 2
- net MISO: track 60.1 -> 0.00 mm, vias 2 -> 0
- net MOSI: track 54.1 -> 0.00 mm, vias 2 -> 0
- net RX_CAM: track 0.00 -> 53.7 mm, vias 0 -> 1
- net BR_DIR: track 27.4 -> 61.8 mm, vias 0 -> 1
- net FL_DIR: track 12.5 -> 30.8 mm
- net 3.3V: track 96.0 -> 83.1 mm
- net TX_BT: track 32.8 -> 43.0 mm
- net BL_DIR: track 23.6 -> 33.5 mm
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