File: elec/eagle/assets/layer3/layer3.sch (EAGLE design)
At the start: 84 parts, among them Q2 AO3402, X1 SM06B-SRSS-TB, Y1 8MHz

Commit message: layer 4 pcb
Parts:
- removed BNO055: (no value), SparkFun-Connectors:CONN_08LOCK
- removed R10, R11: 4.7k, SparkFun-Resistors:4.7KOHM-0603-1/10W-1%
Connections:
- removed net MISO: TEENSY4.D12/MISO, U$8.MISO
- removed net MOSI: TEENSY4.D11/MOSI, U$8.MOSI
- removed net SCK: TEENSY4.D13/SCK/LED, U$8.SCLK
- removed net SCL0_TEE: TEENSY4.D17/A3/SDA1, U$8.TXD/SCL
- removed net SDA0_TEE: TEENSY4.D16/A2/SCL1, U$8.RXD/SDA
- removed net SS: TEENSY4.D10/CS, U$8.SSEL
- new net RX_CAM: TEENSY4.D17/A3/SDA1, U$8.RXD/SDA
- new net TX_CAM: TEENSY4.D16/A2/SCL1, U$8.TXD/SCL
- net 3.3V: no longer R10.2, R11.2
- net 3V3_SWITCH: no longer BNO055.8
- net BL_DIR: now also TEENSY4.D11/MOSI; no longer TEENSY4.D26/A12
- net BR_DIR: now also TEENSY4.D6; no longer TEENSY4.D27/A13
- net ESC_LV: now also TEENSY4.D9; no longer TEENSY4.D33/MCLK2
- net FL_DIR: now also TEENSY4.D12/MISO; no longer TEENSY4.D24/A10
- net FR_DIR: now also TEENSY4.D13/SCK/LED; no longer TEENSY4.D25/A11
- net GND: no longer BNO055.7
- net RX_BT: now also TEENSY4.D14/A0; no longer TEENSY4.D29/TX7
- net SCL1: no longer BNO055.5, R11.1
- net SDA1: no longer BNO055.6, R10.1
- net SERVO_LV: now also TEENSY4.D10/CS; no longer TEENSY4.D30/CRX3
- net TX_BT: now also TEENSY4.D15/A1; no longer TEENSY4.D28/RX7
